File: genesis-controller-hat.kicad_sch (KiCad schematic)
At the start: 3 parts, among them J1 GPIO, J2 DE9_Socket_MountingHoles, J3 DE9_Socket_MountingHoles

Commit message: Correct J2/J3 from female DB9 sockets to male DB9 pins
A real Sega Genesis controller's cable ends in a female DB9 connector, so
the HAT needs male ports to receive it -- the opposite of what had been
designed. This was never checked against a datasheet, photo, or real
hardware until physically verified against two real controllers (original
and third-party). Corrected schematic symbols (DE9_Socket_MountingHoles ->
DE9_Pins_MountingHoles) and PCB footprints (DSUB-9_Socket_Horizontal_... ->
DSUB-9_Pins_Horizontal_..., same overhang/mounting-hole variant).

A male DB9's physical pin order mirrors a female one's left-to-right, which
broke the earlier GPIO reassignment's careful non-crossing correspondence
(verified: the resulting conflict graph had 65 edges and wasn't
2-colorable). Re-derived a new GPIO assignment matched to the male
connector's actual pin order (see
docs/reviews/2026-07-22-pinmap-reassignment.md for the full analysis);
GPIO12/23 move to spare, GPIO9/11 move out of spare. Verified zero
crossings computationally before implementing.

J2/J3 re-placed (mounting holes also mirror position) and fully re-routed,
including activating J1's previously-unwired GPIO9/GPIO11 pins and freeing
GPIO12/GPIO23. scripts/check_pinmap.py updated for the mirrored pin
offsets. Final state: ERC 0/0, DRC 4 errors/0 warnings (only +3V3's
structurally-unavoidable long diagonal remains, down from 26 crossings in
the first routing attempt after the gender fix).

Co-Authored-By: Claude Sonnet 5 <noreply@anthropic.com>
Parts:
- J2, J3: value DE9_Socket_MountingHoles -> DE9_Pins_MountingHoles; symbol Connector:DE9_Socket_MountingHoles -> Connector:DE9_Pins_MountingHoles
Connections:
- net GPIO10/SPI0.MOSI: now also J2.4; no longer J2.1
- net GPIO13/PWM1: now also J3.3; no longer J3.2
- net GPIO16: now also J3.4; no longer J3.6
- net GPIO17: now also J2.6; no longer J2.4
- net GPIO24: now also J2.3; no longer J2.6
- net GPIO26: now also J3.9; no longer J3.1
- net GPIO27: now also J2.2; no longer J2.3
- net GPIO4/GPCLK0: now also J2.1; no longer J2.9
- net GPIO5: now also J3.2; no longer J3.4
- net GPIO6: now also J3.7; no longer J3.3
- net GPIO7/SPI0.CE1: now also J3.6; no longer J3.9
- net GPIO9/SPI0.MISO: now reaches J1.21 (Pin_21)
- net GPIO9/SPI0.MISO: now also J2.9
- net GPIO11/SPI0.SCLK: now reaches J1.23 (Pin_23)
- net GPIO11/SPI0.SCLK: now also J3.1
- net GPIO12/PWM0: no longer names the net of J1.32 (Pin_32)
- net GPIO12/PWM0: no longer J3.7
- net GPIO23: no longer names the net of J1.16 (Pin_16)
- net GPIO23: no longer J2.2
Changed lines of the file:
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@@
-	)
-	(no_connect
-		(at 60.96 55.88)
 	)
 	(no_connect
@@
 		(at 73.66 60.96)
 	)
-	(no_connect
-		(at 60.96 53.34)
-	)
 	(wire
 		(pts
@@
 	(wire
 		(pts
-			(xy 73.66 45.72)
-			(xy 100.33 45.72)
-		)
-		(stroke
-			(width 0)
-			(type solid)
-		)
-	)
-	(wire
-		(pts
 			(xy 58.42 76.2)
 			(xy 58.42 80.01)
@@
 	(wire
 		(pts
-			(xy 73.66 66.04)
-			(xy 100.33 66.04)
-		)
-		(stroke
-			(width 0)
-			(type solid)
-		)
-	)
-	(wire
-		(pts
 			(xy 58.42 76.2)
 			(xy 60.96 76.2)
@@
 	)
 	(label "GPIO22"
-		(at 43.18 251.46 0)
-		(effects
-			(font
-				(size 1.27 1.27)
-			)
-			(justify left bottom)
-		)
-	)
-	(label "GPIO10{slash}SPI0.MOSI"
-		(at 43.18 243.84 0)
+		(at 43.18 256.53999999999996 0)
+		(effects
+			(font
+				(size 1.27 1.27)
+			)
+			(justify left bottom)
+		)
+	)
+	(label "GPIO4{slash}GPCLK0"
+		(at 43.18 264.15999999999997 0)
 		(effects
 			(font
@@
 		)
 	)
-	(label "GPIO23"
-		(at 100.33 45.72 180)
-		(effects
-			(font
-				(size 1.27 1.27)
-			)
-			(justify right bottom)
-		)
-	)
 	(label "GPIO4{slash}GPCLK0"
 		(at 31.75 35.56 0)
@@
 		)
 	)
-	(label "GPIO5"
-		(at 93.98 259.08 0)
-		(effects
-			(font
-				(size 1.27 1.27)
-			)
-			(justify left bottom)
-		)
-	)
-	(label "GPIO26"
-		(at 93.98 243.84 0)
+	(label "GPIO16"
+		(at 93.98 248.92000000000002 0)
+		(effects
+			(font
+				(size 1.27 1.27)
+			)
+			(justify left bottom)
+		)
+	)
+	(label "GPIO11{slash}SPI0.SCLK"
+		(at 93.98 264.15999999999997 0)
 		(effects
 			(font
@@
 		)
 	)
-	(label "GPIO17"
-		(at 43.18 259.08 0)
+	(label "GPIO10{slash}SPI0.MOSI"
+		(at 43.18 248.92000000000002 0)
 		(effects
 			(font
@@
 		)
 	)
-	(label "GPIO4{slash}GPCLK0"
-		(at 43.18 261.62 0)
+	(label "GPIO9{slash}SPI0.MISO"
+		(at 43.18 246.38 0)
 		(effects
 			(font
@@
 		)
 	)
-	(label "GPIO13{slash}PWM1"
-		(at 93.98 248.92 0)
+	(label "GPIO5"
+		(at 93.98 259.08000000000004 0)
 		(effects
 			(font
@@
 		)
 	)
+	(label "GPIO26"
+		(at 93.98 246.38 0)
+		(effects
+			(font
+				(size 1.27 1.27)
+			)
+			(justify left bottom)
+		)
+	)
+	(label "GPIO24"
+		(at 43.18 254.0 0)
+		(effects
+			(font
+				(size 1.27 1.27)
+			)
+			(justify left bottom)
+		)
+	)
 	(label "GPIO7{slash}SPI0.CE1"
 		(at 93.98 261.62 0)
@@
 		)
 	)
-	(label "GPIO27"
-		(at 43.18 254 0)
-		(effects
-			(font
-				(size 1.27 1.27)
-			)
-			(justify left bottom)
-		)
-	)
-	(label "GPIO16"
-		(at 93.98 246.38 0)
-		(effects
-			(font
-				(size 1.27 1.27)
-			)
-			(justify left bottom)
-		)
-	)
 	(label "GPIO17"
 		(at 31.75 40.64 0)
@@
 		)
 	)
-	(label "GPIO12{slash}PWM0"
-		(at 93.98 251.46 0)
-		(effects
-			(font
-				(size 1.27 1.27)
-			)
-			(justify left bottom)
-		)
-	)
 	(label "GPIO6"
-		(at 93.98 254 0)
-		(effects
-			(font
-				(size 1.27 1.27)
-			)
-			(justify left bottom)
-		)
-	)
-	(label "GPIO12{slash}PWM0"
-		(at 100.33 66.04 180)
-		(effects
-			(font
-				(size 1.27 1.27)
-			)
-			(justify right bottom)
+		(at 93.98 256.53999999999996 0)
+		(effects
+			(font
+				(size 1.27 1.27)
+			)
+			(justify left bottom)
+		)
+	)
+	(label "GPIO13{slash}PWM1"
+		(at 93.98 254.0 0)
+		(effects
+			(font
+				(size 1.27 1.27)
+			)
+			(justify left bottom)
 		)
 	)
@@
 		)
 	)
-	(label "GPIO23"
-		(at 43.18 248.92 0)
-		(effects
-			(font
-				(size 1.27 1.27)
-			)
-			(justify left bottom)
-		)
-	)
-	(label "GPIO24"
-		(at 43.18 246.38 0)
+	(label "GPIO27"
+		(at 43.18 259.08000000000004 0)
+		(effects
+			(font
+				(size 1.27 1.27)
+			)
+			(justify left bottom)
+		)
+	)
+	(label "GPIO17"
+		(at 43.18 261.62 0)
 		(effects
 			(font
@@
 	)
 	(symbol
-		(lib_id "Connector:DE9_Socket_MountingHoles")
+		(lib_id "Connector:DE9_Pins_MountingHoles")
 		(at 101.6 254 0)
 		(unit 1)
@@
 			)
 		)
-		(property "Value" "DE9_Socket_MountingHoles"
+		(property "Value" "DE9_Pins_MountingHoles"
 			(at 101.6 238.125 0)
 			(show_name no)
@@
 	(symbol
 		(lib_id "power:+3.3V")
-		(at 93.98 264.16 0)
+		(at 93.98 243.83999999999997 0)
 		(unit 1)
 		(body_style 1)
@@
 	)
 	(symbol
-		(lib_id "Connector:DE9_Socket_MountingHoles")
+		(lib_id "Connector:DE9_Pins_MountingHoles")
 		(at 50.8 254 0)
 		(unit 1)
@@
 			)
 		)
-		(property "Value" "DE9_Socket_MountingHoles"
+		(property "Value" "DE9_Pins_MountingHoles"
 			(at 50.8 238.125 0)
 			(show_name no)
@@
 	(symbol
 		(lib_id "power:+3.3V")
-		(at 43.18 264.16 0)
+		(at 43.18 243.83999999999997 0)
 		(unit 1)
 		(body_style 1)
@@
 	(symbol
 		(lib_id "power:GND")
-		(at 93.98 256.54 0)
+		(at 93.98 251.45999999999998 0)
 		(unit 1)
 		(body_style 1)
@@
 	(symbol
 		(lib_id "power:GND")
-		(at 43.18 256.54 0)
+		(at 43.18 251.45999999999998 0)
 		(unit 1)
 		(body_style 1)
@@
 		)
 	)
+	(no_connect
+		(at 73.66 45.72)
+	)
+	(no_connect
+		(at 73.66 66.04)
+	)
+	(wire
+		(pts
+			(xy 60.96 53.34)
+			(xy 31.75 53.34)
+		)
+		(stroke
+			(width 0)
+			(type default)
+		)
+	)
+	(label "GPIO9{slash}SPI0.MISO"
+		(at 31.75 53.34 0)
+		(effects
+			(font
+				(size 1.27 1.27)
+			)
+			(justify left bottom)
+		)
+	)
+	(wire
+		(pts
+			(xy 60.96 55.88)
+			(xy 31.75 55.88)
+		)
+		(stroke
+			(width 0)
+			(type default)
+		)
+	)
+	(label "GPIO11{slash}SPI0.SCLK"
+		(at 31.75 55.88 0)
+		(effects
+			(font
+				(size 1.27 1.27)
+			)
+			(justify left bottom)
+		)
+	)
