File: genesis-controller-hat.kicad_sch (KiCad schematic)
At the start: 3 parts, among them J1 GPIO, J2 DE9_Pins_MountingHoles, J3 DE9_Pins_MountingHoles

Commit message: Fix stale Footprint property on J2/J3 -- ERC still 0/0
Schematic Footprint property still pointed at the pre-rework
DSUB-9_Socket_Vertical footprint (wrong gender, wrong orientation),
even though the actual PCB footprint and lib_id were already correct.
Left as-is, it would silently revert J2/J3 on the next "Update PCB
from Schematic".
Parts:
- J2, J3: footprint Connector_Dsub:DSUB-9_Socket_Vertical_P2.77x2.84mm_MountingHoles -> Connector_Dsub:DSUB-9_Pins_Horizontal_P2.77x2.84mm_EdgePinOffset7.70mm_Housed_MountingHolesOffset9.12mm
Changed lines of the file:
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@@
 			)
 		)
-		(property "Footprint" "Connector_Dsub:DSUB-9_Socket_Vertical_P2.77x2.84mm_MountingHoles"
+		(property "Footprint" "Connector_Dsub:DSUB-9_Pins_Horizontal_P2.77x2.84mm_EdgePinOffset7.70mm_Housed_MountingHolesOffset9.12mm"
 			(at 101.6 254 0)
 			(hide yes)
@@
 			)
 		)
-		(property "Footprint" "Connector_Dsub:DSUB-9_Socket_Vertical_P2.77x2.84mm_MountingHoles"
+		(property "Footprint" "Connector_Dsub:DSUB-9_Pins_Horizontal_P2.77x2.84mm_EdgePinOffset7.70mm_Housed_MountingHolesOffset9.12mm"
 			(at 50.8 254 0)
 			(hide yes)
